Commit message: [WIP]Add MujocoKinovaGen3Cable.

File: robo_manip_baselines/envs/assets/common/robots/kinovagen3/kinovagen3.urdf (robot description, URDF)
Before this commit: robot gen3, 12 links, 11 joints
Links:
- removed link left_base_link
- removed link left_bicep_link
- removed link left_bracelet_link
- removed link left_camera_color_frame
- removed link left_camera_depth_frame
- removed link left_camera_link
- removed link left_end_effector_link
- removed link left_forearm_link
- removed link left_shoulder_link
- removed link left_spherical_wrist_1_link
- removed link left_spherical_wrist_2_link
- removed link left_tool_frame
- added link base_link, mass 1.697; collision mesh filename=package://kortex_description/arms/gen3/6dof/meshes/base_lin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; visual mesh filename=package://kortex_description/arms/gen3/6dof/meshes/base_lin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
- added link bicep_link, mass 1.262; collision mesh filename=package://kortex_description/arms/gen3/6dof/meshes/bicep_li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; visual mesh filename=package://kortex_description/arms/gen3/6dof/meshes/bicep_li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
- added link bracelet_link, mass 0.5; collision mesh filename=package://kortex_description/arms/gen3/6dof/meshes/bracelet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; visual mesh filename=package://kortex_description/arms/gen3/6dof/meshes/bracelet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
- added link end_effector_link
- added link forearm_link, mass 0.93; collision mesh filename=package://kortex_description/arms/gen3/6dof/meshes/forearm_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; visual mesh filename=package://kortex_description/arms/gen3/6dof/meshes/forearm_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
- added link shoulder_link, mass 1.377; collision mesh filename=package://kortex_description/arms/gen3/6dof/meshes/shoulder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; visual mesh filename=package://kortex_description/arms/gen3/6dof/meshes/shoulder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
- added link spherical_wrist_1_link, mass 0.6781; collision mesh filename=package://kortex_description/arms/gen3/6dof/meshes/spherica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; visual mesh filename=package://kortex_description/arms/gen3/6dof/meshes/spherica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
- added link spherical_wrist_2_link, mass 0.678; collision mesh filename=package://kortex_description/arms/gen3/6dof/meshes/spherica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; visual mesh filename=package://kortex_description/arms/gen3/6dof/meshes/spherica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
Joints:
- removed joint left_camera_module
- removed joint left_color_module
- removed joint left_depth_module
- removed joint left_end_effector
- removed joint left_joint_1
- removed joint left_joint_2
- removed joint left_joint_3
- removed joint left_joint_4
- removed joint left_joint_5
- removed joint left_joint_6
- removed joint left_tool_frame_joint
- added joint end_effector: type revolute, parent bracelet_link, child end_effector_link, origin xyz=0 0 0 rpy=0 0 0, limit lower=-3.1101767270538954 upper=3.1101767270538954 effort=20 velocity=3.14
- added joint joint_1: type revolute, parent base_link, child shoulder_link, origin xyz=0 0 0.15643 rpy=-3.1416 0.0 0.0, axis 0 0 1, limit effort=39 velocity=1.3963
- added joint joint_2: type revolute, parent shoulder_link, child bicep_link, origin xyz=0 0.005375 -0.12838 rpy=1.5708 0.0 0.0, axis 0 0 1, limit lower=-2.24 upper=2.24 effort=39 velocity=1.3963
- added joint joint_3: type revolute, parent bicep_link, child forearm_link, origin xyz=0 -0.41 0 rpy=3.1416 0 0, axis 0 0 1, limit lower=-2.57 upper=2.57 effort=39 velocity=1.3963
- added joint joint_4: type revolute, parent forearm_link, child spherical_wrist_1_link, origin xyz=0 0.20843 -0.006375 rpy=1.5708 0.0 0.0, axis 0 0 1, limit effort=9 velocity=1.2218
- added joint joint_5: type revolute, parent spherical_wrist_1_link, child spherical_wrist_2_link, origin xyz=0 -0.00017505 -0.10593 rpy=-1.5708 0.0 0.0, axis 0 0 1, limit lower=-2.09 upper=2.09 effort=9 velocity=1.2218
- added joint joint_6: type revolute, parent spherical_wrist_2_link, child bracelet_link, origin xyz=0 0.10593 -0.00017505 rpy=1.5708 0.0 0.0, axis 0 0 1, limit effort=9 velocity=1.2218

Commit message: Fix urdf

File: robo_manip_baselines/envs/assets/common/robots/kinovagen3/kinovagen3.urdf (robot description, URDF)
Before this commit: robot gen3, 8 links, 7 joints
Links:
- removed link bicep_link
- added link half_arm_1_link, mass 1.1636; collision mesh filename=package://kortex_description/arms/gen3/7dof/meshes/half_arm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; visual mesh filename=package://kortex_description/arms/gen3/7dof/meshes/half_arm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
- added link half_arm_2_link, mass 1.1636; collision mesh filename=package://kortex_description/arms/gen3/7dof/meshes/half_arm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; visual mesh filename=package://kortex_description/arms/gen3/7dof/meshes/half_arm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
- link base_link: geometry collision mesh filename=package://kortex_description/arms/gen3/7dof/meshes/base_lin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; visual mesh filename=package://kortex_description/arms/gen3/7dof/meshes/base_lin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
- link bracelet_link: mass 0.5 -> 0.5006; geometry collision mesh filename=package://kortex_description/arms/gen3/7dof/meshes/bracelet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; visual mesh filename=package://kortex_description/arms/gen3/7dof/meshes/bracelet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
- link forearm_link: mass 0.93 -> 0.9302; geometry collision mesh filename=package://kortex_description/arms/gen3/7dof/meshes/forearm_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; visual mesh filename=package://kortex_description/arms/gen3/7dof/meshes/forearm_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
- link shoulder_link: mass 1.377 -> 1.3773; geometry collision mesh filename=package://kortex_description/arms/gen3/7dof/meshes/shoulder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; visual mesh filename=package://kortex_description/arms/gen3/7dof/meshes/shoulder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
- link spherical_wrist_1_link: geometry collision mesh filename=package://kortex_description/arms/gen3/7dof/meshes/spherica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; visual mesh filename=package://kortex_description/arms/gen3/7dof/meshes/spherica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
- link spherical_wrist_2_link: mass 0.678 -> 0.6781; geometry collision mesh filename=package://kortex_description/arms/gen3/7dof/meshes/spherica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; visual mesh filename=package://kortex_description/arms/gen3/7dof/meshes/spherica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
Joints:
- added joint joint_7: type revolute, parent spherical_wrist_2_link, child bracelet_link, origin xyz=0 -0.10593 -0.00017505 rpy=-1.5708 -5.5511E-17 9.6396E-17, axis 0 0 1, limit effort=9 velocity=1.2218
- joint end_effector: limit lower=-3.1101767270538954 upper=3.1101767270538954 effort=20 velocity=3.14 -> (none); type revolute -> fixed
- joint joint_1: origin xyz=0 0 0.15643 rpy=-3.1416 0.0 0.0 -> xyz=0 0 0.15643 rpy=3.1416 2.7629E-18 -4.9305E-36
- joint joint_2: child bicep_link -> half_arm_1_link; origin xyz=0 0.005375 -0.12838 rpy=1.5708 0.0 0.0 -> xyz=0 0.005375 -0.12838 rpy=1.5708 2.1343E-17 -1.1102E-16
- joint joint_3: child forearm_link -> half_arm_2_link; limit lower=-2.57 upper=2.57 effort=39 velocity=1.3963 -> effort=39 velocity=1.3963; origin xyz=0 -0.41 0 rpy=3.1416 0 0 -> xyz=0 -0.21038 -0.006375 rpy=-1.5708 1.2326E-32 -2.9122E-16; parent bicep_link -> half_arm_1_link
- joint joint_4: child spherical_wrist_1_link -> forearm_link; limit effort=9 velocity=1.2218 -> lower=-2.57 upper=2.57 effort=39 velocity=1.3963; origin xyz=0 0.20843 -0.006375 rpy=1.5708 0.0 0.0 -> xyz=0 0.006375 -0.21038 rpy=1.5708 -6.6954E-17 -1.6653E-16; parent forearm_link -> half_arm_2_link
- joint joint_5: child spherical_wrist_2_link -> spherical_wrist_1_link; limit lower=-2.09 upper=2.09 effort=9 velocity=1.2218 -> effort=9 velocity=1.2218; origin xyz=0 -0.00017505 -0.10593 rpy=-1.5708 0.0 0.0 -> xyz=0 -0.20843 -0.006375 rpy=-1.5708 2.2204E-16 -6.373E-17; parent spherical_wrist_1_link -> forearm_link
- joint joint_6: child bracelet_link -> spherical_wrist_2_link; limit effort=9 velocity=1.2218 -> lower=-2.09 upper=2.09 effort=9 velocity=1.2218; origin xyz=0 0.10593 -0.00017505 rpy=1.5708 0.0 0.0 -> xyz=0 0.00017505 -0.10593 rpy=1.5708 9.2076E-28 -8.2157E-15; parent spherical_wrist_2_link -> spherical_wrist_1_link

Commit message: [envs] Update KinovaGen3.

File: robo_manip_baselines/envs/assets/common/robots/kinovagen3/kinovagen3.urdf (robot description, URDF)
Before this commit: robot gen3, 9 links, 8 joints
Joints:
- joint joint_1: limit effort=39 velocity=1.3963 -> lower=-6.28 upper=6.28 effort=39 velocity=1.3963
- joint joint_3: limit effort=39 velocity=1.3963 -> lower=-6.28 upper=6.28 effort=39 velocity=1.3963
- joint joint_5: limit effort=9 velocity=1.2218 -> lower=-6.28 upper=6.28 effort=9 velocity=1.2218
- joint joint_7: limit effort=9 velocity=1.2218 -> lower=-6.28 upper=6.28 effort=9 velocity=1.2218
