Commit message: add board task

File: robo_manip_baselines/envs/assets/tacto/objects/cylinder/rod.urdf (robot description, URDF)
Before this commit: robot rod, 1 links, 0 joints
Links:
- link rod: mass 0.2 -> 0.05; geometry collision cylinder length=0.30 radius=0.0058; visual cylinder length=0.30 radius=0.006
