Commit message: Update TactoSawyerInsertEnv.

File: robo_manip_baselines/envs/assets/tacto/objects/insert/board.urdf (robot description, URDF)
Before this commit: robot cube, 1 links, 0 joints
Links:
- removed link cube
- added link board, mass 0.2; collision box size=.005 .05 .29; visual box size=.005 .05 .29

File: robo_manip_baselines/envs/assets/tacto/objects/insert/box.urdf (robot description, URDF)
Before this commit: robot cylinder, 1 links, 0 joints
Links:
- removed link cylinder
- added link box, mass 1.0; collision mesh filename=meshes/vhacd_box.obj; visual mesh filename=meshes/box.obj

File: robo_manip_baselines/envs/assets/tacto/objects/insert/cube.urdf (robot description, URDF)
Before this commit: robot board, 1 links, 0 joints
Links:
- removed link board
- added link cube, mass 0.2; collision box size=.03 .03 .136; visual box size=.03 .03 .136
